Commit message: 换为新版realman程序

File: rm_robot/rm_65_description/urdf/rm_65.urdf.xacro (robot description, xacro)
@@ -1,29 +1,221 @@
-<?xml version="1.0" ?>
-<robot name="rm_65" xmlns:xacro="http://www.ros.org/wiki/xacro">
+<?xml version="1.0" encoding="utf-8"?>
+<robot name="rm_65_with_wheeltec" xmlns:xacro="http://www.ros.org/wiki/xacro">
 <xacro:include filename="$(find rm_65_description)/urdf/rm_65.transmission.xacro"/>
 <xacro:include filename="$(find rm_65_description)/urdf/rm_65.gazebo.xacro"/>
-<!-- <xacro:include filename="$(find rm_65_description)/urdf/common.gazebo.xacro"/> -->
-<!-- Inertial matrix -->
-<xacro:macro name="inertial_matrix" params="mass">
-<inertial>
-    <mass value="${mass}" />
-    <inertia ixx="1.0" ixy="0.0" ixz="0.0" iyy="0.5" iyz="0.0" izz="1.0" />
-</inertial>
-</xacro:macro>
-  <link
-    name="base_link">
-    <inertial>
-      <origin
-        xyz="0.000364099338239377 -0.000180492589223954 0.0523748178864983"
+  <!-- =========================== Wheeltec Mobile Base =========================== -->
+  <link name="base_link_wheeltec">
+    <inertial>
+      <origin xyz="0 0 0.0975" rpy="0 0 0"/>
+      <mass value="5.0"/>
+      <inertia
+        ixx="0.1"
+        ixy="0.0"
+        ixz="0.0"
+        iyy="0.1"
+        iyz="0.0"
+        izz="0.1"/>
+    </inertial>
+    <visual>
+      <origin xyz="0 0 0.0975" rpy="0 0 0" />
+      <geometry>
+        <box size="0.27 0.185 0.055"/>
+      </geometry>
+      <material name="white">
+        <color rgba="1 1 1 1"/>
+      </material>
+    </visual>
+    <collision>
+      <origin xyz="0 0 0.0975" rpy="0 0 0" />
+      <geometry>
+        <box size="0.27 0.185 0.055"/>
+      </geometry>
+    </collision>
+  </link>
+  <!-- 添加Gazebo物理属性 -->
+  <gazebo reference="base_link_wheeltec">
+    <mu1 value="0.5"/>
+    <mu2 value="0.5"/>
+    <kp value="1000000.0"/>
+    <kd value="100.0"/>
+  </gazebo>
+  <!-- 前左轮 -->
+  <joint name="left_front_joint" type="continuous">
+    <origin xyz="0.085 0.09 0.0375" rpy="1.57 0 0"/>
+    <parent link="base_link_wheeltec"/>
+    <child link="left_front_link"/>
+    <axis xyz="0 1 0"/>
+  </joint>
+  <link name="left_front_link">
+    <inertial>
+      <origin xyz="0 0 0" rpy="0 0 0"/>
+      <mass value="0.5"/>
+      <inertia
+        ixx="0.0005"
+        ixy="0.0"
+        ixz="0.0"
+        iyy="0.001"
+        iyz="0.0"
+        izz="0.0005"/>
+    </inertial>
+    <visual>
+      <origin xyz="0 0 0" rpy="0 0 0" />
+      <geometry>
+        <cylinder radius="0.0375" length="0.03"/>
+      </geometry>
+      <material name="black">
+        <color rgba="0 0 0 1"/>
+      </material>
+    </visual>
+    <collision>
+      <origin xyz="0 0 0" rpy="0 0 0" />
+      <geometry>
+        <cylinder radius="0.0375" length="0.03"/>
+      </geometry>
+    </collision>
+  </link>
+  <!-- 前右轮 -->
+  <joint name="right_front_joint" type="continuous">
+    <origin xyz="0.085 -0.09 0.0375" rpy="1.57 0 0"/>
+    <parent link="base_link_wheeltec"/>
+    <child link="right_front_link"/>
+    <axis xyz="0 1 0"/>
+  </joint>
+  <link name="right_front_link">
+    <inertial>
+      <origin xyz="0 0 0" rpy="0 0 0"/>
+      <mass value="0.5"/>
+      <inertia
+        ixx="0.0005"
+        ixy="0.0"
+        ixz="0.0"
+        iyy="0.001"
+        iyz="0.0"
+        izz="0.0005"/>
+    </inertial>
+    <visual>
+      <origin xyz="0 0 0" rpy="0 0 0" />
+      <geometry>
+        <cylinder radius="0.0375" length="0.03"/>
+      </geometry>
+      <material name="black">
+        <color rgba="0 0 0 1"/>
+      </material>
+    </visual>
+    <collision>
+      <origin xyz="0 0 0" rpy="0 0 0" />
+      <geometry>
+        <cylinder radius="0.0375" length="0.03"/>
+      </geometry>
+    </collision>
+  </link>
+  <!-- 后左轮 -->
+  <joint name="left_wheel_joint" type="continuous">
+    <origin xyz="-0.085 0.09 0.0375" rpy="1.57 0 0"/>
+    <parent link="base_link_wheeltec"/>
+    <child link="left_wheel_link"/>
+    <axis xyz="0 1 0"/>
+  </joint>
+  <link name="left_wheel_link">
+    <inertial>
+      <origin xyz="0 0 0" rpy="0 0 0"/>
+      <mass value="0.5"/>
+      <inertia
+        ixx="0.0005"
+        ixy="0.0"
+        ixz="0.0"
+        iyy="0.001"
+        iyz="0.0"
+        izz="0.0005"/>
+    </inertial>
+    <visual>
+      <origin xyz="0 0 0" rpy="0 0 0" />
+      <geometry>
+        <cylinder radius="0.0375" length="0.03"/>
+      </geometry>
+      <material name="black">
+        <color rgba="0 0 0 1"/>
+      </material>
+    </visual>
+    <collision>
+      <origin xyz="0 0 0" rpy="0 0 0" />
+      <geometry>
+        <cylinder radius="0.0375" length="0.03"/>
+      </geometry>
+    </collision>
+  </link>
+  <!-- 后右轮 -->
+  <joint name="right_wheel_joint" type="continuous">
+    <origin xyz="-0.085 -0.09 0.0375" rpy="1.57 0 0"/>
+    <parent link="base_link_wheeltec"/>
+    <child link="right_wheel_link"/>
+    <axis xyz="0 1 0"/>
+  </joint>
+  <link name="right_wheel_link">
+    <inertial>
+      <origin xyz="0 0 0" rpy="0 0 0"/>
+      <mass value="0.5"/>
+      <inertia
+        ixx="0.0005"
+        ixy="0.0"
+        ixz="0.0"
+        iyy="0.001"
+        iyz="0.0"
+        izz="0.0005"/>
+    </inertial>
+    <visual>
+      <origin xyz="0 0 0" rpy="0 0 0" />
+      <geometry>
+        <cylinder radius="0.0375" length="0.03"/>
+      </geometry>
+      <material name="black">
+        <color rgba="0 0 0 1"/>
+      </material>
+    </visual>
+    <collision>
+      <origin xyz="0 0 0" rpy="0 0 0" />
+      <geometry>
+        <cylinder radius="0.0375" length="0.03"/>
+      </geometry>
+    </collision>
+  </link>
+  <!-- 为轮子添加Gazebo插件 -->
+  <gazebo reference="left_front_link">
+    <mu1 value="1.0"/>
+    <mu2 value="1.0"/>
+  </gazebo>
+  <gazebo reference="right_front_link">
+    <mu1 value="1.0"/>
+    <mu2 value="1.0"/>
+  </gazebo>
+  <gazebo reference="left_wheel_link">
+    <mu1 value="1.0"/>
+    <mu2 value="1.0"/>
+  </gazebo>
+  <gazebo reference="right_wheel_link">
+    <mu1 value="1.0"/>
+    <mu2 value="1.0"/>
+  </gazebo>
+  <!-- =========================== RM-65 Arm Base (放在Wheeltec上方20cm) =========================== -->
+  <!-- 连接关节：从Wheeltec底盘到RM-65基座 -->
+  <joint name="wheeltec_to_arm_joint" type="fixed">
+    <origin xyz="0 0 0.4" rpy="0 0 3.1415926"/>
+    <parent link="base_link_wheeltec"/>
+    <child link="base_link"/>
+  </joint>
+  <!-- RM-65机械臂的base_link -->
+  <link name="base_link">
+    <inertial>
+      <origin
+        xyz="-0.000433277303987328 -3.54664423471128E-05 0.0599427668933796"
         rpy="0 0 0" />
       <mass
-        value="14" />
-      <inertia
-        ixx="0.000737277875726733"
-        ixy="1.52768076655905E-06"
-        ixz="-1.75138967359717E-05"
-        iyy="0.000723643543181375"
-        iyz="-8.08320706906158E-07"
-        izz="0.000487026166065825" />
+        value="0.841070778135659" />
+      <inertia
+        ixx="0.0017261110801622"
+        ixy="2.52746264980217E-06"
+        ixz="-3.67690303614961E-05"
+        iyy="0.00170987405835604"
+        iyz="1.67996364994424E-06"
+        izz="0.000904023422915791" />
     </inertial>
     <visual>
@@ -57,27 +249,28 @@
     <kd value="1.0"/>
   </gazebo>
+  <!-- =========================== RM-65 Arm Links and Joints =========================== -->
   <link
     name="Link1">
     <inertial>
       <origin
-        xyz="-1.79862733952242E-05 -0.0216004812887538 0.0719258896443856"
+        xyz="1.2226305431569E-08 0.0211079974844683 -0.0251854220842269"
         rpy="0 0 0" />
       <mass
-        value="0.200843839724735" />
-      <inertia
-        ixx="0.000531136984021332"
-        ixy="-4.32776127280478E-07"
-        ixz="1.04793272362077E-06"
-        iyy="0.000497444611373595"
-        iyz="0.000106254355496355"
-        izz="0.000282103590137435" />
-    </inertial>
-    <visual>
-      <origin
-        xyz="0 0 0"
-        rpy="0 0 0" />
-      <geometry>
-        <mesh
-          filename="package://rm_65_description/meshes/Link1.STL" />
+        value="0.593563443690403" />
+      <inertia
+        ixx="0.00126614120341847"
+        ixy="-1.294980943835E-08"
+        ixz="-9.80120923066996E-09"
+        iyy="0.00118168178300364"
+        iyz="-0.00021121727444415"
+        izz="0.00056135241627747" />
+    </inertial>
+    <visual>
+      <origin
+        xyz="0 0 0"
+        rpy="0 0 0" />
+      <geometry>
+        <mesh
+          filename="package://rm_65_description/meshes/link1.STL" />
       </geometry>
       <material
@@ -93,5 +286,5 @@
       <geometry>
         <mesh
-          filename="package://rm_65_description/meshes/Link1.STL" />
+          filename="package://rm_65_description/meshes/link1.STL" />
       </geometry>
     </collision>
@@ -101,6 +294,6 @@
     type="revolute">
     <origin
-      xyz="0.00019414 0.0001 0.138"
-      rpy="-2.3944E-16 0 3.1416" />
+      xyz="0 0 0.2405"
+      rpy="0 0 0" />
     <parent
       link="base_link" />
@@ -110,7 +303,7 @@
       xyz="0 0 1" />
     <limit
-      lower="-3.14"
-      upper="3.14"
-      effort="300"
+      lower="-3.1"
+      upper="3.1"
+      effort="60"
       velocity="3.14" />
 	<dynamics damping="50" friction="1"/>
@@ -120,23 +313,23 @@
     <inertial>
       <origin
-        xyz="0.133181684940056 -4.09216469913973E-05 0.0184216581306229"
+        xyz="0.152256463426163 4.75383656106654E-07 -0.00620260383607792"
         rpy="0 0 0" />
       <mass
-        value="0.321307361964397" />
-      <inertia
-        ixx="0.000440014028766832"
-        ixy="5.6579315252598E-07"
-        ixz="-0.000654853772254918"
-        iyy="0.00298539844077015"
-        iyz="1.20748806355071E-07"
-        izz="0.00284806640328522" />
-    </inertial>
-    <visual>
-      <origin
-        xyz="0 0 0"
-        rpy="0 0 0" />
-      <geometry>
-        <mesh
-          filename="package://rm_65_description/meshes/Link2.STL" />
+        value="0.864175046869043" />
+      <inertia
+        ixx="0.00089150298478414"
+        ixy="-2.23268489334765E-08"
+        ixz="0.00156246461035015"
+        iyy="0.00733754343083901"
+        iyz="6.28110889329165E-09"
+        izz="0.00697869103915473" />
+    </inertial>
+    <visual>
+      <origin
+        xyz="0 0 0"
+        rpy="0 0 0" />
+      <geometry>
+        <mesh
+          filename="package://rm_65_description/meshes/link2.STL" />
       </geometry>
       <material
@@ -152,5 +345,5 @@
       <geometry>
         <mesh
-          filename="package://rm_65_description/meshes/Link2.STL" />
+          filename="package://rm_65_description/meshes/link2.STL" />
       </geometry>
     </collision>
@@ -160,5 +353,5 @@
     type="revolute">
     <origin
-      xyz="0 0.016171 0.1012"
+      xyz="0 0 0"
       rpy="1.5708 -1.5708 0" />
     <parent
@@ -167,9 +360,9 @@
       link="Link2" />
     <axis
-      xyz="0 0 -1" />
+      xyz="0 0 1" />
     <limit
-      lower="-2.269"
-      upper="2.269"
-      effort="300"
+      lower="-2.268"
+      upper="2.268"
+      effort="60"
       velocity="3.14" />
 	<dynamics damping="50" friction="1"/>
@@ -179,23 +372,23 @@
     <inertial>
       <origin
-        xyz="-3.56690328818382E-06 -0.0512866037910138 2.10951876323563E-05"
+        xyz="5.05312670989961E-06 -0.0595925663694732 0.010569069212336"
         rpy="0 0 0" />
       <mass
-        value="0.102772515618803" />
-      <inertia
-        ixx="0.000236471825455939"
-        ixy="-2.85439143488268E-09"
-        ixz="-4.04883470632046E-10"
-        iyy="7.36858171850124E-05"
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
Commit message: 修改srdf

File: rm_robot/rm_65_description/urdf/rm_65.urdf.xacro (robot description, xacro)
@@ -1,639 +1,664 @@
 <?xml version="1.0" encoding="utf-8"?>
-<robot name="rm_65_with_wheeltec" xmlns:xacro="http://www.ros.org/wiki/xacro">
+<robot name="rm_65" xmlns:xacro="http://www.ros.org/wiki/xacro">
 <xacro:include filename="$(find rm_65_description)/urdf/rm_65.transmission.xacro"/>
 <xacro:include filename="$(find rm_65_description)/urdf/rm_65.gazebo.xacro"/>
-  <!-- =========================== Wheeltec Mobile Base =========================== -->
-  <link name="base_link_wheeltec">
-    <inertial>
-      <origin xyz="0 0 0.0975" rpy="0 0 0"/>
-      <mass value="5.0"/>
-      <inertia
-        ixx="0.1"
-        ixy="0.0"
-        ixz="0.0"
-        iyy="0.1"
-        iyz="0.0"
-        izz="0.1"/>
-    </inertial>
-    <visual>
-      <origin xyz="0 0 0.0975" rpy="0 0 0" />
-      <geometry>
-        <box size="0.27 0.185 0.055"/>
-      </geometry>
-      <material name="white">
-        <color rgba="1 1 1 1"/>
-      </material>
-    </visual>
-    <collision>
-      <origin xyz="0 0 0.0975" rpy="0 0 0" />
-      <geometry>
-        <box size="0.27 0.185 0.055"/>
-      </geometry>
-    </collision>
-  </link>
-  <!-- 添加Gazebo物理属性 -->
-  <gazebo reference="base_link_wheeltec">
-    <mu1 value="0.5"/>
-    <mu2 value="0.5"/>
-    <kp value="1000000.0"/>
-    <kd value="100.0"/>
-  </gazebo>
-  <!-- 前左轮 -->
-  <joint name="left_front_joint" type="continuous">
-    <origin xyz="0.085 0.09 0.0375" rpy="1.57 0 0"/>
-    <parent link="base_link_wheeltec"/>
-    <child link="left_front_link"/>
-    <axis xyz="0 1 0"/>
-  </joint>
-  <link name="left_front_link">
-    <inertial>
-      <origin xyz="0 0 0" rpy="0 0 0"/>
-      <mass value="0.5"/>
-      <inertia
-        ixx="0.0005"
-        ixy="0.0"
-        ixz="0.0"
-        iyy="0.001"
-        iyz="0.0"
-        izz="0.0005"/>
-    </inertial>
-    <visual>
-      <origin xyz="0 0 0" rpy="0 0 0" />
-      <geometry>
-        <cylinder radius="0.0375" length="0.03"/>
-      </geometry>
-      <material name="black">
-        <color rgba="0 0 0 1"/>
-      </material>
-    </visual>
-    <collision>
-      <origin xyz="0 0 0" rpy="0 0 0" />
-      <geometry>
-        <cylinder radius="0.0375" length="0.03"/>
-      </geometry>
-    </collision>
-  </link>
-  <!-- 前右轮 -->
-  <joint name="right_front_joint" type="continuous">
-    <origin xyz="0.085 -0.09 0.0375" rpy="1.57 0 0"/>
-    <parent link="base_link_wheeltec"/>
-    <child link="right_front_link"/>
-    <axis xyz="0 1 0"/>
-  </joint>
-  <link name="right_front_link">
-    <inertial>
-      <origin xyz="0 0 0" rpy="0 0 0"/>
-      <mass value="0.5"/>
-      <inertia
-        ixx="0.0005"
-        ixy="0.0"
-        ixz="0.0"
-        iyy="0.001"
-        iyz="0.0"
-        izz="0.0005"/>
-    </inertial>
-    <visual>
-      <origin xyz="0 0 0" rpy="0 0 0" />
-      <geometry>
-        <cylinder radius="0.0375" length="0.03"/>
-      </geometry>
-      <material name="black">
-        <color rgba="0 0 0 1"/>
-      </material>
-    </visual>
-    <collision>
-      <origin xyz="0 0 0" rpy="0 0 0" />
-      <geometry>
-        <cylinder radius="0.0375" length="0.03"/>
-      </geometry>
-    </collision>
-  </link>
-  <!-- 后左轮 -->
-  <joint name="left_wheel_joint" type="continuous">
-    <origin xyz="-0.085 0.09 0.0375" rpy="1.57 0 0"/>
-    <parent link="base_link_wheeltec"/>
-    <child link="left_wheel_link"/>
-    <axis xyz="0 1 0"/>
-  </joint>
-  <link name="left_wheel_link">
-    <inertial>
-      <origin xyz="0 0 0" rpy="0 0 0"/>
-      <mass value="0.5"/>
-      <inertia
-        ixx="0.0005"
-        ixy="0.0"
-        ixz="0.0"
-        iyy="0.001"
-        iyz="0.0"
-        izz="0.0005"/>
-    </inertial>
-    <visual>
-      <origin xyz="0 0 0" rpy="0 0 0" />
-      <geometry>
-        <cylinder radius="0.0375" length="0.03"/>
-      </geometry>
-      <material name="black">
-        <color rgba="0 0 0 1"/>
-      </material>
-    </visual>
-    <collision>
-      <origin xyz="0 0 0" rpy="0 0 0" />
-      <geometry>
-        <cylinder radius="0.0375" length="0.03"/>
-      </geometry>
-    </collision>
-  </link>
-  <!-- 后右轮 -->
-  <joint name="right_wheel_joint" type="continuous">
-    <origin xyz="-0.085 -0.09 0.0375" rpy="1.57 0 0"/>
-    <parent link="base_link_wheeltec"/>
-    <child link="right_wheel_link"/>
-    <axis xyz="0 1 0"/>
-  </joint>
-  <link name="right_wheel_link">
-    <inertial>
-      <origin xyz="0 0 0" rpy="0 0 0"/>
-      <mass value="0.5"/>
-      <inertia
-        ixx="0.0005"
-        ixy="0.0"
-        ixz="0.0"
-        iyy="0.001"
-        iyz="0.0"
-        izz="0.0005"/>
-    </inertial>
-    <visual>
-      <origin xyz="0 0 0" rpy="0 0 0" />
-      <geometry>
-        <cylinder radius="0.0375" length="0.03"/>
-      </geometry>
-      <material name="black">
-        <color rgba="0 0 0 1"/>
-      </material>
-    </visual>
-    <collision>
-      <origin xyz="0 0 0" rpy="0 0 0" />
-      <geometry>
-        <cylinder radius="0.0375" length="0.03"/>
-      </geometry>
-    </collision>
-  </link>
-  <!-- 为轮子添加Gazebo插件 -->
-  <gazebo reference="left_front_link">
-    <mu1 value="1.0"/>
-    <mu2 value="1.0"/>
-  </gazebo>
-  <gazebo reference="right_front_link">
-    <mu1 value="1.0"/>
-    <mu2 value="1.0"/>
-  </gazebo>
-  <gazebo reference="left_wheel_link">
-    <mu1 value="1.0"/>
-    <mu2 value="1.0"/>
-  </gazebo>
-  <gazebo reference="right_wheel_link">
-    <mu1 value="1.0"/>
-    <mu2 value="1.0"/>
-  </gazebo>
-  <!-- =========================== RM-65 Arm Base (放在Wheeltec上方20cm) =========================== -->
-  <!-- 连接关节：从Wheeltec底盘到RM-65基座 -->
-  <joint name="wheeltec_to_arm_joint" type="fixed">
-    <origin xyz="0 0 0.4" rpy="0 0 3.1415926"/>
-    <parent link="base_link_wheeltec"/>
-    <child link="base_link"/>
-  </joint>
-  <!-- RM-65机械臂的base_link -->
-  <link name="base_link">
-    <inertial>
-      <origin
-        xyz="-0.000433277303987328 -3.54664423471128E-05 0.0599427668933796"
-        rpy="0 0 0" />
-      <mass
-        value="0.841070778135659" />
-      <inertia
-        ixx="0.0017261110801622"
-        ixy="2.52746264980217E-06"
-        ixz="-3.67690303614961E-05"
-        iyy="0.00170987405835604"
-        iyz="1.67996364994424E-06"
-        izz="0.000904023422915791" />
-    </inertial>
-    <visual>
-      <origin
-        xyz="0 0 0"
-        rpy="0 0 0" />
-      <geometry>
-        <mesh
-          filename="package://rm_65_description/meshes/base_link.STL" />
-      </geometry>
-      <material
-        name="">
-        <color
-          rgba="1 1 1 1" />
-      </material>
-    </visual>
-    <collision>
-      <origin
-        xyz="0 0 0"
-        rpy="0 0 0" />
-      <geometry>
-        <mesh
-          filename="package://rm_65_description/meshes/base_link.STL" />
-      </geometry>
-    </collision>
-  </link>
-  <gazebo reference="base_link">
-    <mu1 value="200000.0"/>
-    <mu2 value="200000.0"/>
-    <kp value="100000000.0"/>
-    <kd value="1.0"/>
-  </gazebo>
-  <!-- =========================== RM-65 Arm Links and Joints =========================== -->
-  <link
-    name="Link1">
-    <inertial>
-      <origin
-        xyz="1.2226305431569E-08 0.0211079974844683 -0.0251854220842269"
-        rpy="0 0 0" />
-      <mass
-        value="0.593563443690403" />
-      <inertia
-        ixx="0.00126614120341847"
-        ixy="-1.294980943835E-08"
-        ixz="-9.80120923066996E-09"
-        iyy="0.00118168178300364"
-        iyz="-0.00021121727444415"
-        izz="0.00056135241627747" />
-    </inertial>
-    <visual>
-      <origin
-        xyz="0 0 0"
-        rpy="0 0 0" />
-      <geometry>
-        <mesh
-          filename="package://rm_65_description/meshes/link1.STL" />
-      </geometry>
-      <material
-        name="">
-        <color
-          rgba="1 1 1 1" />
-      </material>
-    </visual>
-    <collision>
-      <origin
-        xyz="0 0 0"
-        rpy="0 0 0" />
-      <geometry>
-        <mesh
-          filename="package://rm_65_description/meshes/link1.STL" />
-      </geometry>
-    </collision>
-  </link>
-  <joint
-    name="joint1"
-    type="revolute">
-    <origin
-      xyz="0 0 0.2405"
-      rpy="0 0 0" />
-    <parent
-      link="base_link" />
-    <child
-      link="Link1" />
-    <axis
-      xyz="0 0 1" />
-    <limit
-      lower="-3.1"
-      upper="3.1"
-      effort="60"
-      velocity="3.14" />
+<!-- =========================== 添加虚拟根链接解决KDL问题 =========================== -->
+<link name="world"/>
+<link name="virtual_base_link">
+  <inertial>
+    <mass value="0.001"/>
+    <inertia ixx="0.000001" ixy="0.0" ixz="0.0" iyy="0.000001" iyz="0.0" izz="0.000001"/>
+  </inertial>
+</link>
+<joint name="world_to_virtual_joint" type="fixed">
+  <parent link="world"/>
+  <child link="virtual_base_link"/>
+  <origin xyz="0 0 0" rpy="0 0 0"/>
+</joint>
+<!-- 修改原来的base_link_wheeltec惯性参数 -->
+<link name="base_link_wheeltec">
+  <!-- 减小惯性参数以避免KDL警告 -->
+  <inertial>
+    <origin xyz="0 0 0.0975" rpy="0 0 0"/>
+    <mass value="0.1"/>  <!-- 减小质量 -->
+    <inertia
+      ixx="0.001"
+      ixy="0.0"
+      ixz="0.0"
+      iyy="0.001"
+      iyz="0.0"
+      izz="0.001"/>
+  </inertial>
+  <visual>
+    <origin xyz="0 0 0.0975" rpy="0 0 0" />
+    <geometry>
+      <box size="0.27 0.185 0.055"/>
+    </geometry>
+    <material name="white">
+      <color rgba="1 1 1 1"/>
+    </material>
+  </visual>
+  <collision>
+    <origin xyz="0 0 0.0975" rpy="0 0 0" />
+    <geometry>
+      <box size="0.27 0.185 0.055"/>
+    </geometry>
+  </collision>
+</link>
+<joint name="virtual_to_wheeltec_joint" type="fixed">
+  <parent link="virtual_base_link"/>
+  <child link="base_link_wheeltec"/>
+  <origin xyz="0 0 0" rpy="0 0 0"/>
+</joint>
+<!-- 添加Gazebo物理属性 -->
+<gazebo reference="base_link_wheeltec">
+  <mu1 value="0.5"/>
+  <mu2 value="0.5"/>
+  <kp value="1000000.0"/>
+  <kd value="100.0"/>
+</gazebo>
+<!-- =========================== Wheeltec Mobile Base =========================== -->
+<!-- 修改轮子关节类型：continuous -> revolute -->
+<!-- 前左轮 -->
+<joint name="left_front_joint" type="revolute">
+  <origin xyz="0.085 0.09 0.0375" rpy="1.57 0 0"/>
+  <parent link="base_link_wheeltec"/>
+  <child link="left_front_link"/>
+  <axis xyz="0 1 0"/>
+  <limit lower="-100" upper="100" effort="10" velocity="10"/>
+</joint>
+<link name="left_front_link">
+  <inertial>
+    <origin xyz="0 0 0" rpy="0 0 0"/>
+    <mass value="0.5"/>
+    <inertia
+      ixx="0.0005"
+      ixy="0.0"
+      ixz="0.0"
+      iyy="0.001"
+      iyz="0.0"
+      izz="0.0005"/>
+  </inertial>
+  <visual>
+    <origin xyz="0 0 0" rpy="0 0 0" />
+    <geometry>
+      <cylinder radius="0.0375" length="0.03"/>
+    </geometry>
+    <material name="black">
+      <color rgba="0 0 0 1"/>
+    </material>
+  </visual>
+  <collision>
+    <origin xyz="0 0 0" rpy="0 0 0" />
+    <geometry>
+      <cylinder radius="0.0375" length="0.03"/>
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