Commit message: 生成简易视点

File: rm_robot/rm_65_description/urdf/rm_65.urdf.xacro (robot description, xacro)
@@ -30,8 +30,8 @@
       <origin xyz="0 0 0.17" rpy="0 0 0" />  <!-- 高度中心：13cm/2=6.5cm -->
       <geometry>
-          <box size="0.5 0.4 0.34"/>  <!-- 长×宽×高：50cm×40cm×13cm -->
+          <box size="0.5 0.4 0.3"/>  <!-- 长×宽×高：50cm×40cm×13cm -->
       </geometry>
       <material name="white">
-          <color rgba="1 1 1 1"/>
+          <color rgba="1 1 0 1"/>
       </material>
   </visual>
@@ -54,5 +54,5 @@
 <!-- 前左轮 -->
 <joint name="left_front_joint" type="revolute">
-  <origin xyz="0.085 0.09 0.0375" rpy="1.57 0 0"/>
+  <origin xyz="0.191 0.201  0.0375" rpy="1.57 0 0"/>
   <parent link="base_link_wheeltec"/>
   <child link="left_front_link"/>
@@ -90,5 +90,5 @@
 <!-- 前右轮 -->
 <joint name="right_front_joint" type="revolute">
-  <origin xyz="0.085 -0.09 0.0375" rpy="1.57 0 0"/>
+  <origin xyz="0.191 -0.201  0.0375" rpy="1.57 0 0"/>
   <parent link="base_link_wheeltec"/>
   <child link="right_front_link"/>
@@ -126,5 +126,5 @@
 <!-- 后左轮 -->
 <joint name="left_wheel_joint" type="revolute">
-  <origin xyz="-0.085 0.09 0.0375" rpy="1.57 0 0"/>
+  <origin xyz="-0.191 0.201  0.0375" rpy="1.57 0 0"/>
   <parent link="base_link_wheeltec"/>
   <child link="left_wheel_link"/>
@@ -162,5 +162,5 @@
 <!-- 后右轮 -->
 <joint name="right_wheel_joint" type="revolute">
-  <origin xyz="-0.085 -0.09 0.0375" rpy="1.57 0 0"/>
+  <origin xyz="-0.191 -0.201  0.0375" rpy="1.57 0 0"/>
   <parent link="base_link_wheeltec"/>
   <child link="right_wheel_link"/>

Commit message: 调整机器人造型

File: rm_robot/rm_65_description/urdf/rm_65.urdf.xacro (robot description, xacro)
@@ -54,5 +54,5 @@
 <!-- 前左轮 -->
 <joint name="left_front_joint" type="revolute">
-  <origin xyz="0.191 0.201  0.0375" rpy="1.57 0 0"/>
+  <origin xyz="0.191 0.202  0.0375" rpy="1.57 0 0"/>
   <parent link="base_link_wheeltec"/>
   <child link="left_front_link"/>
@@ -90,5 +90,5 @@
 <!-- 前右轮 -->
 <joint name="right_front_joint" type="revolute">
-  <origin xyz="0.191 -0.201  0.0375" rpy="1.57 0 0"/>
+  <origin xyz="0.191 -0.202  0.0375" rpy="1.57 0 0"/>
   <parent link="base_link_wheeltec"/>
   <child link="right_front_link"/>
@@ -126,5 +126,5 @@
 <!-- 后左轮 -->
 <joint name="left_wheel_joint" type="revolute">
-  <origin xyz="-0.191 0.201  0.0375" rpy="1.57 0 0"/>
+  <origin xyz="-0.191 0.202  0.0375" rpy="1.57 0 0"/>
   <parent link="base_link_wheeltec"/>
   <child link="left_wheel_link"/>
@@ -162,5 +162,5 @@
 <!-- 后右轮 -->
 <joint name="right_wheel_joint" type="revolute">
-  <origin xyz="-0.191 -0.201  0.0375" rpy="1.57 0 0"/>
+  <origin xyz="-0.191 -0.202  0.0375" rpy="1.57 0 0"/>
   <parent link="base_link_wheeltec"/>
   <child link="right_wheel_link"/>

Commit message: 在rm_65.urdf.xacro中加入了相机和大轮子

File: rm_robot/rm_65_description/urdf/rm_65.urdf.xacro (robot description, xacro)
@@ -4,4 +4,20 @@
 <xacro:include filename="$(find rm_65_description)/urdf/rm_65.gazebo.xacro"/>
 <!-- =========================== 添加虚拟根链接解决KDL问题 =========================== -->
+<xacro:property name="wheel_radius" value="0.05" />  <!-- 轮子半径 -->
+<xacro:property name="wheel_length" value="0.03" />
+<!-- KINECT DK 相机 -->
+<xacro:property name="kinect_dk_box_width" value="0.1" />
+<xacro:property name="kinect_dk_box_length" value="0.14" />
+<xacro:property name="kinect_dk_box_height" value="0.04" />
+<xacro:property name="kinect_pose_h" value="0.035" />
+<material name="yellow">
+  <color rgba="1 1 0 1"/> </material>
+<material name="red">
+  <color rgba="1 0.2 0.2 0.5"/> </material>
+<material name="blue">
+  <color rgba="0.2 0.2 1  0.5"/> </material>
+<material name="black">
+  <color rgba="0 0 0 1"/>
+</material>
 <!-- 修改原来的base_link_wheeltec惯性参数 -->
 <link name="base_link_wheeltec">
@@ -33,5 +49,5 @@
       </geometry>
       <material name="white">
-          <color rgba="1 1 0 1"/>
+          <color rgba="0.7 0.7 0.7 1"/>    <!-- 底盘颜色 -->
       </material>
   </visual>
@@ -54,5 +70,5 @@
 <!-- 前左轮 -->
 <joint name="left_front_joint" type="revolute">
-  <origin xyz="0.191 0.202  0.0375" rpy="1.57 0 0"/>
+  <origin xyz="0.191 0.202  ${wheel_radius}" rpy="1.57 0 0"/>
   <parent link="base_link_wheeltec"/>
   <child link="left_front_link"/>
@@ -75,5 +91,5 @@
     <origin xyz="0 0 0" rpy="0 0 0" />
     <geometry>
-      <cylinder radius="0.0375" length="0.03"/>
+      <cylinder radius="${wheel_radius}" length="0.03"/>
     </geometry>
     <material name="black">
@@ -84,5 +100,5 @@
     <origin xyz="0 0 0" rpy="0 0 0" />
     <geometry>
-      <cylinder radius="0.0375" length="0.03"/>
+      <cylinder radius="${wheel_radius}" length="0.03"/>
     </geometry>
   </collision>
@@ -90,5 +106,5 @@
 <!-- 前右轮 -->
 <joint name="right_front_joint" type="revolute">
-  <origin xyz="0.191 -0.202  0.0375" rpy="1.57 0 0"/>
+  <origin xyz="0.191 -0.202  ${wheel_radius}" rpy="1.57 0 0"/>
   <parent link="base_link_wheeltec"/>
   <child link="right_front_link"/>
@@ -111,5 +127,5 @@
     <origin xyz="0 0 0" rpy="0 0 0" />
     <geometry>
-      <cylinder radius="0.0375" length="0.03"/>
+      <cylinder radius="${wheel_radius}" length="0.03"/>
     </geometry>
     <material name="black">
@@ -120,5 +136,5 @@
     <origin xyz="0 0 0" rpy="0 0 0" />
     <geometry>
-      <cylinder radius="0.0375" length="0.03"/>
+      <cylinder radius="${wheel_radius}" length="0.03"/>
     </geometry>
   </collision>
@@ -126,5 +142,5 @@
 <!-- 后左轮 -->
 <joint name="left_wheel_joint" type="revolute">
-  <origin xyz="-0.191 0.202  0.0375" rpy="1.57 0 0"/>
+  <origin xyz="-0.191 0.202  ${wheel_radius}" rpy="1.57 0 0"/>
   <parent link="base_link_wheeltec"/>
   <child link="left_wheel_link"/>
@@ -147,5 +163,5 @@
     <origin xyz="0 0 0" rpy="0 0 0" />
     <geometry>
-      <cylinder radius="0.0375" length="0.03"/>
+      <cylinder radius="${wheel_radius}" length="0.03"/>
     </geometry>
     <material name="black">
@@ -156,5 +172,5 @@
     <origin xyz="0 0 0" rpy="0 0 0" />
     <geometry>
-      <cylinder radius="0.0375" length="0.03"/>
+      <cylinder radius="${wheel_radius}" length="0.03"/>
     </geometry>
   </collision>
@@ -162,5 +178,5 @@
 <!-- 后右轮 -->
 <joint name="right_wheel_joint" type="revolute">
-  <origin xyz="-0.191 -0.202  0.0375" rpy="1.57 0 0"/>
+  <origin xyz="-0.191 -0.202  ${wheel_radius}" rpy="1.57 0 0"/>
   <parent link="base_link_wheeltec"/>
   <child link="right_wheel_link"/>
@@ -183,5 +199,5 @@
     <origin xyz="0 0 0" rpy="0 0 0" />
     <geometry>
-      <cylinder radius="0.0375" length="0.03"/>
+      <cylinder radius="${wheel_radius}" length="0.03"/>
     </geometry>
     <material name="black">
@@ -192,5 +208,5 @@
     <origin xyz="0 0 0" rpy="0 0 0" />
     <geometry>
-      <cylinder radius="0.0375" length="0.03"/>
+      <cylinder radius="${wheel_radius}" length="0.03"/>
     </geometry>
   </collision>
@@ -620,4 +636,35 @@
     velocity="3.92" />
 	<dynamics damping="50" friction="1"/>
+</joint>
+<!-- kinect dk 相机 -->
+<link name="kinect_dk_camera_link">
+  <visual>
+    <origin xyz="0 0 0" rpy="0 0 0" />
+    <geometry>
+      <box size="${kinect_dk_box_width} ${kinect_dk_box_length} ${kinect_dk_box_height}" />
+    </geometry>
+    <material name="blue"/>
+  </visual>
+  <collision>
+    <origin xyz="0 0 0" rpy="0 0 0" />
+    <geometry>
+      <box size="${kinect_dk_box_width} ${kinect_dk_box_length} ${kinect_dk_box_height}" />
+    </geometry>
+  </collision>
+  <inertial>
+    <origin xyz="0 0 0" rpy="0 0 0" />
+    <mass value="0.5" /> <inertia
+      ixx="${0.5 * (kinect_dk_box_length*kinect_dk_box_length + kinect_dk_box_height*kinect_dk_box_height)}"
+      ixy="0.0"
+      ixz="0.0"
+      iyy="${0.5 * (kinect_dk_box_width*kinect_dk_box_width + kinect_dk_box_height*kinect_dk_box_height)}"
+      iyz="0.0"
+      izz="${0.5 * (kinect_dk_box_width*kinect_dk_box_width + kinect_dk_box_length*kinect_dk_box_length)}" />
+  </inertial>
+</link>
+<joint name="kinect_dk_camera_joint" type="fixed">
+  <origin xyz="0  0.0 ${kinect_pose_h}" rpy="0 0 0"/>
+  <parent link="Link6"/>
+  <child link="kinect_dk_camera_link"/>
 </joint>
 <!-- =========================== Transmission and Control =========================== -->
