Commit message: 修改了urdf文件,记得改回来; 修改了view planning SE3文件,准备加入根据机器人位置判断功能

File: rm_robot/rm_65_description/urdf/mini_4wd_robot加入rm但是底盘动不了了.urdf (robot description, URDF)
Before this commit: robot wheeltec_robot, 5 links, 4 joints
Links:
- removed link base_link
- added link base_link_wheeltec; visual box size=0.27 0.185 0.055
Joints:
- joint left_front_joint: parent base_link -> base_link_wheeltec
- joint left_wheel_joint: parent base_link -> base_link_wheeltec
- joint right_front_joint: parent base_link -> base_link_wheeltec
- joint right_wheel_joint: parent base_link -> base_link_wheeltec

File: rm_robot/rm_65_description/urdf/rm_65.urdf(自制底盘).xacro (robot description, xacro)
@@ -4,16 +4,20 @@
 <xacro:include filename="$(find rm_65_description)/urdf/rm_65.gazebo.xacro"/>
 <!-- =========================== 添加虚拟根链接解决KDL问题 =========================== -->
-<link name="world"/>
-<link name="virtual_base_link">
-  <inertial>
-    <mass value="0.001"/>
-    <inertia ixx="0.000001" ixy="0.0" ixz="0.0" iyy="0.000001" iyz="0.0" izz="0.000001"/>
-  </inertial>
-</link>
-<joint name="world_to_virtual_joint" type="fixed">
-  <parent link="world"/>
-  <child link="virtual_base_link"/>
-  <origin xyz="0 0 0" rpy="0 0 0"/>
-</joint>
+<xacro:property name="wheel_radius" value="0.05" />  <!-- 轮子半径 -->
+<xacro:property name="wheel_length" value="0.03" />
+<!-- KINECT DK 相机 -->
+<xacro:property name="kinect_dk_box_width" value="0.1" />
+<xacro:property name="kinect_dk_box_length" value="0.14" />
+<xacro:property name="kinect_dk_box_height" value="0.04" />
+<xacro:property name="kinect_pose_h" value="0.035" />
+<material name="yellow">
+  <color rgba="1 1 0 1"/> </material>
+<material name="red">
+  <color rgba="1 0.2 0.2 0.5"/> </material>
+<material name="blue">
+  <color rgba="0.2 0.2 1  0.5"/> </material>
+<material name="black">
+  <color rgba="0 0 0 1"/>
+</material>
 <!-- 修改原来的base_link_wheeltec惯性参数 -->
 <link name="base_link_wheeltec">
@@ -30,5 +34,5 @@
       izz="0.001"/>
   </inertial>
-  <visual>
+  <!-- <visual>
     <origin xyz="0 0 0.0975" rpy="0 0 0" />
     <geometry>
@@ -38,4 +42,13 @@
       <color rgba="1 1 1 1"/>
     </material>
+  </visual> -->
+   <visual>
+      <origin xyz="0 0 0.17" rpy="0 0 0" />  <!-- 高度中心：13cm/2=6.5cm -->
+      <geometry>
+          <box size="0.5 0.4 0.3"/>  <!-- 长×宽×高：50cm×40cm×13cm -->
+      </geometry>
+      <material name="white">
+          <color rgba="0.7 0.7 0.7 1"/>    <!-- 底盘颜色 -->
+      </material>
   </visual>
   <collision>
@@ -46,9 +59,4 @@
   </collision>
 </link>
-<joint name="virtual_to_wheeltec_joint" type="fixed">
-  <parent link="virtual_base_link"/>
-  <child link="base_link_wheeltec"/>
-  <origin xyz="0 0 0" rpy="0 0 0"/>
-</joint>
 <!-- 添加Gazebo物理属性 -->
 <gazebo reference="base_link_wheeltec">
@@ -62,5 +70,5 @@
 <!-- 前左轮 -->
 <joint name="left_front_joint" type="revolute">
-  <origin xyz="0.085 0.09 0.0375" rpy="1.57 0 0"/>
+  <origin xyz="0.191 0.202  ${wheel_radius}" rpy="1.57 0 0"/>
   <parent link="base_link_wheeltec"/>
   <child link="left_front_link"/>
@@ -83,5 +91,5 @@
     <origin xyz="0 0 0" rpy="0 0 0" />
     <geometry>
-      <cylinder radius="0.0375" length="0.03"/>
+      <cylinder radius="${wheel_radius}" length="0.03"/>
     </geometry>
     <material name="black">
@@ -92,5 +100,5 @@
     <origin xyz="0 0 0" rpy="0 0 0" />
     <geometry>
-      <cylinder radius="0.0375" length="0.03"/>
+      <cylinder radius="${wheel_radius}" length="0.03"/>
     </geometry>
   </collision>
@@ -98,5 +106,5 @@
 <!-- 前右轮 -->
 <joint name="right_front_joint" type="revolute">
-  <origin xyz="0.085 -0.09 0.0375" rpy="1.57 0 0"/>
+  <origin xyz="0.191 -0.202  ${wheel_radius}" rpy="1.57 0 0"/>
   <parent link="base_link_wheeltec"/>
   <child link="right_front_link"/>
@@ -119,5 +127,5 @@
     <origin xyz="0 0 0" rpy="0 0 0" />
     <geometry>
-      <cylinder radius="0.0375" length="0.03"/>
+      <cylinder radius="${wheel_radius}" length="0.03"/>
     </geometry>
     <material name="black">
@@ -128,5 +136,5 @@
     <origin xyz="0 0 0" rpy="0 0 0" />
     <geometry>
-      <cylinder radius="0.0375" length="0.03"/>
+      <cylinder radius="${wheel_radius}" length="0.03"/>
     </geometry>
   </collision>
@@ -134,5 +142,5 @@
 <!-- 后左轮 -->
 <joint name="left_wheel_joint" type="revolute">
-  <origin xyz="-0.085 0.09 0.0375" rpy="1.57 0 0"/>
+  <origin xyz="-0.191 0.202  ${wheel_radius}" rpy="1.57 0 0"/>
   <parent link="base_link_wheeltec"/>
   <child link="left_wheel_link"/>
@@ -155,5 +163,5 @@
     <origin xyz="0 0 0" rpy="0 0 0" />
     <geometry>
-      <cylinder radius="0.0375" length="0.03"/>
+      <cylinder radius="${wheel_radius}" length="0.03"/>
     </geometry>
     <material name="black">
@@ -164,5 +172,5 @@
     <origin xyz="0 0 0" rpy="0 0 0" />
     <geometry>
-      <cylinder radius="0.0375" length="0.03"/>
+      <cylinder radius="${wheel_radius}" length="0.03"/>
     </geometry>
   </collision>
@@ -170,5 +178,5 @@
 <!-- 后右轮 -->
 <joint name="right_wheel_joint" type="revolute">
-  <origin xyz="-0.085 -0.09 0.0375" rpy="1.57 0 0"/>
+  <origin xyz="-0.191 -0.202  ${wheel_radius}" rpy="1.57 0 0"/>
   <parent link="base_link_wheeltec"/>
   <child link="right_wheel_link"/>
@@ -191,5 +199,5 @@
     <origin xyz="0 0 0" rpy="0 0 0" />
     <geometry>
-      <cylinder radius="0.0375" length="0.03"/>
+      <cylinder radius="${wheel_radius}" length="0.03"/>
     </geometry>
     <material name="black">
@@ -200,5 +208,5 @@
     <origin xyz="0 0 0" rpy="0 0 0" />
     <geometry>
-      <cylinder radius="0.0375" length="0.03"/>
+      <cylinder radius="${wheel_radius}" length="0.03"/>
     </geometry>
   </collision>
@@ -223,5 +231,5 @@
 <!-- =========================== RM-65 Arm Base =========================== -->
 <joint name="wheeltec_to_arm_joint" type="fixed">
-  <origin xyz="0 0 0.4" rpy="0 0 3.1415926"/>
+  <origin xyz="0 0 0.34" rpy="0 0 3.1415926"/>
   <parent link="base_link_wheeltec"/>
   <child link="base_link"/>
@@ -628,4 +636,35 @@
     velocity="3.92" />
 	<dynamics damping="50" friction="1"/>
+</joint>
+<!-- kinect dk 相机 -->
+<link name="kinect_dk_camera_link">
+  <visual>
+    <origin xyz="0 0 0" rpy="0 0 0" />
+    <geometry>
+      <box size="${kinect_dk_box_width} ${kinect_dk_box_length} ${kinect_dk_box_height}" />
+    </geometry>
+    <material name="blue"/>
+  </visual>
+  <collision>
+    <origin xyz="0 0 0" rpy="0 0 0" />
+    <geometry>
+      <box size="${kinect_dk_box_width} ${kinect_dk_box_length} ${kinect_dk_box_height}" />
+    </geometry>
+  </collision>
+  <inertial>
+    <origin xyz="0 0 0" rpy="0 0 0" />
+    <mass value="0.5" /> <inertia
+      ixx="${0.5 * (kinect_dk_box_length*kinect_dk_box_length + kinect_dk_box_height*kinect_dk_box_height)}"
+      ixy="0.0"
+      ixz="0.0"
+      iyy="${0.5 * (kinect_dk_box_width*kinect_dk_box_width + kinect_dk_box_height*kinect_dk_box_height)}"
+      iyz="0.0"
+      izz="${0.5 * (kinect_dk_box_width*kinect_dk_box_width + kinect_dk_box_length*kinect_dk_box_length)}" />
+  </inertial>
+</link>
+<joint name="kinect_dk_camera_joint" type="fixed">
+  <origin xyz="0  0.0 ${kinect_pose_h}" rpy="0 0 0"/>
+  <parent link="Link6"/>
+  <child link="kinect_dk_camera_link"/>
 </joint>
 <!-- =========================== Transmission and Control =========================== -->

File: rm_robot/rm_65_description/urdf/rm_65.urdf.xacro (robot description, xacro)
@@ -1,7 +1,9 @@
 <?xml version="1.0" encoding="utf-8"?>
-<robot name="rm_65" xmlns:xacro="http://www.ros.org/wiki/xacro">
+<robot name="rm_65_combined" xmlns:xacro="http://www.ros.org/wiki/xacro">
 <xacro:include filename="$(find rm_65_description)/urdf/rm_65.transmission.xacro"/>
 <xacro:include filename="$(find rm_65_description)/urdf/rm_65.gazebo.xacro"/>
-<!-- =========================== 添加虚拟根链接解决KDL问题 =========================== -->
+<xacro:property name="wheel_radius" value="0.05" />
+<xacro:property name="wheel_length" value="0.03" />
+<xacro:property name="kinect_pose_h" value="0.035" />
 <xacro:property name="wheel_radius" value="0.05" />  <!-- 轮子半径 -->
 <xacro:property name="wheel_length" value="0.03" />
@@ -11,630 +13,243 @@
 <xacro:property name="kinect_dk_box_height" value="0.04" />
 <xacro:property name="kinect_pose_h" value="0.035" />
-<material name="yellow">
-  <color rgba="1 1 0 1"/> </material>
-<material name="red">
-  <color rgba="1 0.2 0.2 0.5"/> </material>
-<material name="blue">
-  <color rgba="0.2 0.2 1  0.5"/> </material>
-<material name="black">
-  <color rgba="0 0 0 1"/>
-</material>
-<!-- 修改原来的base_link_wheeltec惯性参数 -->
+<!-- 材料定义 -->
+<material name="yellow"><color rgba="1 1 0 1"/></material>
+<material name="white"><color rgba="1 1 1 1"/></material>
+<material name="black"><color rgba="0 0 0 1"/></material>
+<material name="blue"><color rgba="0.2 0.2 1 0.5"/></material>
+<material name="red"><color rgba="1 0.2 0.2 0.5"/></material> <!-- 从原文件补充 -->
+<!-- 虚拟根链接 -->
+<link name="base_footprint"/>
+<joint name="base_footprint_joint" type="fixed">
+  <parent link="base_footprint"/>
+  <child link="base_link_wheeltec"/>
+  <origin xyz="0 0 0" rpy="0 0 0"/>
+</joint>
+<!-- 移动底盘 -->
 <link name="base_link_wheeltec">
-  <!-- 减小惯性参数以避免KDL警告 -->
   <inertial>
     <origin xyz="0 0 0.0975" rpy="0 0 0"/>
-    <mass value="0.1"/>  <!-- 减小质量 -->
-    <inertia
-      ixx="0.001"
-      ixy="0.0"
-      ixz="0.0"
-      iyy="0.001"
-      iyz="0.0"
-      izz="0.001"/>
-  </inertial>
-  <!-- <visual>
-    <origin xyz="0 0 0.0975" rpy="0 0 0" />
-    <geometry>
-      <box size="0.27 0.185 0.055"/>
-    </geometry>
-    <material name="white">
-      <color rgba="1 1 1 1"/>
-    </material>
-  </visual> -->
-   <visual>
-      <origin xyz="0 0 0.17" rpy="0 0 0" />  <!-- 高度中心：13cm/2=6.5cm -->
-      <geometry>
-          <box size="0.5 0.4 0.3"/>  <!-- 长×宽×高：50cm×40cm×13cm -->
-      </geometry>
-      <material name="white">
-          <color rgba="0.7 0.7 0.7 1"/>    <!-- 底盘颜色 -->
-      </material>
-  </visual>
-  <collision>
-    <origin xyz="0 0 0.0975" rpy="0 0 0" />
-    <geometry>
-      <box size="0.27 0.185 0.055"/>
-    </geometry>
-  </collision>
-</link>
-<!-- 添加Gazebo物理属性 -->
-<gazebo reference="base_link_wheeltec">
-  <mu1 value="0.5"/>
-  <mu2 value="0.5"/>
-  <kp value="1000000.0"/>
-  <kd value="100.0"/>
-</gazebo>
-<!-- =========================== Wheeltec Mobile Base =========================== -->
-<!-- 修改轮子关节类型：continuous -> revolute -->
-<!-- 前左轮 -->
-<joint name="left_front_joint" type="revolute">
-  <origin xyz="0.191 0.202  ${wheel_radius}" rpy="1.57 0 0"/>
-  <parent link="base_link_wheeltec"/>
-  <child link="left_front_link"/>
-  <axis xyz="0 1 0"/>
-  <limit lower="-100" upper="100" effort="10" velocity="10"/>
-</joint>
-<link name="left_front_link">
-  <inertial>
-    <origin xyz="0 0 0" rpy="0 0 0"/>
-    <mass value="0.5"/>
-    <inertia
-      ixx="0.0005"
-      ixy="0.0"
-      ixz="0.0"
-      iyy="0.001"
-      iyz="0.0"
-      izz="0.0005"/>
-  </inertial>
-  <visual>
-    <origin xyz="0 0 0" rpy="0 0 0" />
-    <geometry>
-      <cylinder radius="${wheel_radius}" length="0.03"/>
-    </geometry>
-    <material name="black">
-      <color rgba="0 0 0 1"/>
-    </material>
-  </visual>
-  <collision>
-    <origin xyz="0 0 0" rpy="0 0 0" />
-    <geometry>
-      <cylinder radius="${wheel_radius}" length="0.03"/>
-    </geometry>
-  </collision>
-</link>
-<!-- 前右轮 -->
-<joint name="right_front_joint" type="revolute">
-  <origin xyz="0.191 -0.202  ${wheel_radius}" rpy="1.57 0 0"/>
-  <parent link="base_link_wheeltec"/>
-  <child link="right_front_link"/>
-  <axis xyz="0 1 0"/>
-  <limit lower="-100" upper="100" effort="10" velocity="10"/>
-</joint>
-<link name="right_front_link">
-  <inertial>
-    <origin xyz="0 0 0" rpy="0 0 0"/>
-    <mass value="0.5"/>
-    <inertia
-      ixx="0.0005"
-      ixy="0.0"
-      ixz="0.0"
-      iyy="0.001"
-      iyz="0.0"
-      izz="0.0005"/>
-  </inertial>
-  <visual>
-    <origin xyz="0 0 0" rpy="0 0 0" />
-    <geometry>
-      <cylinder radius="${wheel_radius}" length="0.03"/>
-    </geometry>
-    <material name="black">
-      <color rgba="0 0 0 1"/>
-    </material>
-  </visual>
-  <collision>
-    <origin xyz="0 0 0" rpy="0 0 0" />
-    <geometry>
-      <cylinder radius="${wheel_radius}" length="0.03"/>
-    </geometry>
-  </collision>
-</link>
-<!-- 后左轮 -->
-<joint name="left_wheel_joint" type="revolute">
-  <origin xyz="-0.191 0.202  ${wheel_radius}" rpy="1.57 0 0"/>
-  <parent link="base_link_wheeltec"/>
-  <child link="left_wheel_link"/>
-  <axis xyz="0 1 0"/>
-  <limit lower="-100" upper="100" effort="10" velocity="10"/>
-</joint>
-<link name="left_wheel_link">
-  <inertial>
-    <origin xyz="0 0 0" rpy="0 0 0"/>
-    <mass value="0.5"/>
-    <inertia
-      ixx="0.0005"
-      ixy="0.0"
-      ixz="0.0"
-      iyy="0.001"
-      iyz="0.0"
-      izz="0.0005"/>
-  </inertial>
-  <visual>
-    <origin xyz="0 0 0" rpy="0 0 0" />
-    <geometry>
-      <cylinder radius="${wheel_radius}" length="0.03"/>
-    </geometry>
-    <material name="black">
-      <color rgba="0 0 0 1"/>
-    </material>
-  </visual>
-  <collision>
-    <origin xyz="0 0 0" rpy="0 0 0" />
-    <geometry>
-      <cylinder radius="${wheel_radius}" length="0.03"/>
-    </geometry>
-  </collision>
-</link>
-<!-- 后右轮 -->
-<joint name="right_wheel_joint" type="revolute">
-  <origin xyz="-0.191 -0.202  ${wheel_radius}" rpy="1.57 0 0"/>
-  <parent link="base_link_wheeltec"/>
-  <child link="right_wheel_link"/>
-  <axis xyz="0 1 0"/>
-  <limit lower="-100" upper="100" effort="10" velocity="10"/>
-</joint>
-<link name="right_wheel_link">
-  <inertial>
-    <origin xyz="0 0 0" rpy="0 0 0"/>
-    <mass value="0.5"/>
-    <inertia
-      ixx="0.0005"
-      ixy="0.0"
-      ixz="0.0"
-      iyy="0.001"
-      iyz="0.0"
-      izz="0.0005"/>
-  </inertial>
-  <visual>
-    <origin xyz="0 0 0" rpy="0 0 0" />
-    <geometry>
-      <cylinder radius="${wheel_radius}" length="0.03"/>
-    </geometry>
-    <material name="black">
-      <color rgba="0 0 0 1"/>
-    </material>
-  </visual>
-  <collision>
-    <origin xyz="0 0 0" rpy="0 0 0" />
-    <geometry>
-      <cylinder radius="${wheel_radius}" length="0.03"/>
-    </geometry>
-  </collision>
-</link>
-<!-- 为轮子添加Gazebo插件 -->
-<gazebo reference="left_front_link">
-  <mu1 value="1.0"/>
-  <mu2 value="1.0"/>
-</gazebo>
-<gazebo reference="right_front_link">
-  <mu1 value="1.0"/>
-  <mu2 value="1.0"/>
-</gazebo>
-<gazebo reference="left_wheel_link">
-  <mu1 value="1.0"/>
-  <mu2 value="1.0"/>
-</gazebo>
-<gazebo reference="right_wheel_link">
-  <mu1 value="1.0"/>
-  <mu2 value="1.0"/>
-</gazebo>
-<!-- =========================== RM-65 Arm Base =========================== -->
+    <mass value="2.0"/>
+    <inertia ixx="0.03" ixy="0.0" ixz="0.0" iyy="0.05" iyz="0.0" izz="0.07"/>
+  </inertial>
+  <visual>
+    <origin xyz="0 0 0.17" rpy="0 0 0" />
+    <geometry><box size="0.5 0.4 0.3"/></geometry>
+    <material name="white"/>
+  </visual>
+  <collision>
+    <origin xyz="0 0 0.17" rpy="0 0 0" />
+    <geometry><box size="0.5 0.4 0.3"/></geometry>
+  </collision>
+</link>
+<!-- 轮子宏定义 -->
+<xacro:macro name="wheel_gen" params="prefix x y">
+  <joint name="${prefix}_joint" type="revolute">
+    <origin xyz="${x} ${y} ${wheel_radius}" rpy="1.57 0 0"/>
+    <parent link="base_link_wheeltec"/>
+    <child link="${prefix}_link"/>
+    <axis xyz="0 1 0"/>
+    <limit lower="-100" upper="100" effort="10" velocity="10"/>
+  </joint>
+  <link name="${prefix}_link">
+    <inertial>
+      <origin xyz="0 0 0" rpy="0 0 0"/>
+      <mass value="0.5"/>
+      <inertia ixx="0.0005" ixy="0.0" ixz="0.0" iyy="0.001" iyz="0.0" izz="0.0005"/>
+    </inertial>
+    <visual>
+      <geometry><cylinder radius="${wheel_radius}" length="${wheel_length}"/></geometry>
+      <material name="black"/>
+    </visual>
+    <collision>
+      <geometry><cylinder radius="${wheel_radius}" length="${wheel_length}"/></geometry>
+    </collision>
+  </link>
+</xacro:macro>
+<xacro:wheel_gen prefix="left_front"  x="0.191"  y="0.202" />
+<xacro:wheel_gen prefix="right_front" x="0.191"  y="-0.202" />
+<xacro:wheel_gen prefix="left_wheel"  x="-0.191" y="0.202" />
+<xacro:wheel_gen prefix="right_wheel" x="-0.191" y="-0.202" />
+<!-- 底盘到机械臂的连接 -->
 <joint name="wheeltec_to_arm_joint" type="fixed">
-  <origin xyz="0 0 0.34" rpy="0 0 3.1415926"/>
+  <origin xyz="0 0 0.32" rpy="0 0 3.1415926"/>
   <parent link="base_link_wheeltec"/>
   <child link="base_link"/>
 </joint>
-<!-- RM-65机械臂的base_link -->
+<!-- RM-65 机械臂 -->
 <link name="base_link">
   <inertial>
-    <origin
-      xyz="-0.000433277303987328 -3.54664423471128E-05 0.0599427668933796"
-      rpy="0 0 0" />
-    <mass
-      value="0.841070778135659" />
-    <inertia
-      ixx="0.0017261110801622"
-      ixy="2.52746264980217E-06"
-      ixz="-3.67690303614961E-05"
-      iyy="0.00170987405835604"
-      iyz="1.67996364994424E-06"
-      izz="0.000904023422915791" />
-  </inertial>
-  <visual>
-    <origin
-      xyz="0 0 0"
-      rpy="0 0 0" />
-    <geometry>
-      <mesh
-        filename="package://rm_65_description/meshes/base_link.STL" />
-    </geometry>
-    <material
-      name="">
-      <color
-        rgba="1 1 1 1" />
-    </material>
-  </visual>
-  <collision>
-    <origin
-      xyz="0 0 0"
-      rpy="0 0 0" />
-    <geometry>
-      <mesh
-        filename="package://rm_65_description/meshes/base_link.STL" />
-    </geometry>
-  </collision>
-</link>
-<gazebo reference="base_link">
-  <mu1 value="200000.0"/>
-  <mu2 value="200000.0"/>
-  <kp value="100000000.0"/>
-  <kd value="1.0"/>
-</gazebo>
-<!-- =========================== RM-65 Arm Links and Joints =========================== -->
-<!-- 保持原有机械臂部分不变 -->
-<link
-  name="Link1">
-  <inertial>
-    <origin
-      xyz="1.2226305431569E-08 0.0211079974844683 -0.0251854220842269"
-      rpy="0 0 0" />
-    <mass
-      value="0.593563443690403" />
-    <inertia
-      ixx="0.00126614120341847"
-      ixy="-1.294980943835E-08"
-      ixz="-9.80120923066996E-09"
-      iyy="0.00118168178300364"
-      iyz="-0.00021121727444415"
-      izz="0.00056135241627747" />
-  </inertial>
-  <visual>
-    <origin
-      xyz="0 0 0"
-      rpy="0 0 0" />
-    <geometry>
-      <mesh
-        filename="package://rm_65_description/meshes/link1.STL" />
-    </geometry>
-    <material
-      name="">
-      <color
-        rgba="1 1 1 1" />
-    </material>
-  </visual>
-  <collision>
-    <origin
-      xyz="0 0 0"
-      rpy="0 0 0" />
-    <geometry>
-      <mesh
-        filename="package://rm_65_description/meshes/link1.STL" />
-    </geometry>
-  </collision>
-</link>
-<joint
-  name="joint1"
-  type="revolute">
-  <origin
-    xyz="0 0 0.2405"
-    rpy="0 0 0" />
-  <parent
-    link="base_link" />
-  <child
-    link="Link1" />
-  <axis
-    xyz="0 0 1" />
-  <limit
-    lower="-3.1"
-    upper="3.1"
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
File: wheeltec/turn_on_wheeltec_robot/urdf/mini_4wd_robot(替换为rm).urdf (robot description, URDF)
Before this commit: robot wheeltec_robot, 5 links, 4 joints
Links:
- removed link base_link
- added link base_link_wheeltec; visual box size=0.5 0.4 0.13
Joints:
- joint left_front_joint: parent base_link -> base_link_wheeltec
- joint left_wheel_joint: parent base_link -> base_link_wheeltec
- joint right_front_joint: parent base_link -> base_link_wheeltec
- joint right_wheel_joint: parent base_link -> base_link_wheeltec
